File: EVA-02/STMboard.kicad_pcb (KiCad board)
At the start: 4 copper layers, 59 parts, among them J1 Screw_Terminal_01x02, J2 USB_B_Micro, J3 Conn_02x05_Odd_Even, J4 Screw_Terminal_01x04, J5 Screw_Terminal_01x05, J6 Screw_Terminal_01x11, J7 Screw_Terminal_01x04, J8 Screw_Terminal_01x05, Q1 AO3401A, SW1 SW_SPDT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

Commit message: Manufactured board files
Parts:
- removed FB2: 100 @ 100MHz, Inductor_SMD:L_0805_2012Metric
- added L2: 39n, Inductor_SMD:L_0402_1005Metric, F.Cu at (130.3, 104.0)
- C10, C11: value 0.1uF -> 100nF
- C13: footprint Capacitor_SMD:C_0201_0603Metric -> Capacitor_SMD:C_0402_1005Metric
- C17: value 100nF -> 1u
- J1: value Screw_Terminal_01x02 -> Screw_Terminal_01x06; footprint TerminalBlock_Phoenix:TerminalBlock_Phoenix_PT-1,5-2-3.5-H_1x02_P3.50mm_Horizontal -> TerminalBlock_Phoenix:TerminalBlock_Phoenix_PT-1,5-6-3.5-H_1x06_P3.50mm_Horizontal
- J3: footprint Connector_PinSocket_1.27mm:PinSocket_2x05_P1.27mm_Vertical_SMD -> Connector_PinHeader_1.27mm:PinHeader_2x05_P1.27mm_Vertical_SMD
- moved H3 393.2 mm to (95.3, 130.5)
- moved J1 381.7 mm to (95.8, 88.7), turned to 270 degrees
- moved SW1 341.9 mm to (136.4, 72.5), turned to 180 degrees
- moved F1 326.9 mm to (121.0, 108.4), turned to 90 degrees
- moved R8 325.6 mm to (108.2, 118.4), turned to 90 degrees
- moved U2 323.2 mm to (114.8, 116.6)
- moved J6 313.8 mm to (106.1, 130.2)
- moved C7 312.4 mm to (119.9, 118.6), turned to 270 degrees
- moved L1 311.1 mm to (110.6, 109.1), turned to 90 degrees
- moved H4 309.8 mm to (95.3, 75.0)
- moved C13 304.8 mm to (114.8, 113.0)
- moved J3 303.8 mm to (175.6, 74.9), turned to 270 degrees
- moved U3 299.0 mm to (117.3, 86.6)
- moved U4 298.0 mm to (167.9, 122.2), turned to 90 degrees
- moved J2 298.0 mm to (168.2, 131.6)
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Connections:
- J5 pad 1: Net-(J5-Pad1) -> +5V
- J5 pad 5: +5V -> Net-(J5-Pad5)
- J8 pad 1: Net-(J8-Pad1) -> +5V
- J8 pad 5: +5V -> Net-(J8-Pad5)
- U1 pad 2: Net-(U1-Pad2) -> PC13
- U1 pad 3: Net-(U1-Pad3) -> PC14
- U1 pad 4: Net-(U1-Pad4) -> PC15
- U1 pad 8: Net-(U1-Pad8) -> PC8
- U5 pad 13: Net-(J5-Pad4) -> Net-(J5-Pad2)
- U5 pad 15: Net-(J5-Pad2) -> Net-(J5-Pad4)
- U5 pad 16: Net-(J5-Pad1) -> Net-(J5-Pad5)
- U6 pad 13: Net-(J8-Pad4) -> Net-(J8-Pad2)
- U6 pad 15: Net-(J8-Pad2) -> Net-(J8-Pad4)
- U6 pad 16: Net-(J8-Pad1) -> Net-(J8-Pad5)
Routing:
- net GND: track 0.00 -> 117.4 mm, vias 0 -> 39
- net +5V: track 0.00 -> 90.8 mm, vias 0 -> 2
- net I2C1_SDA: track 0.00 -> 57.6 mm, vias 0 -> 1
- net NRST: track 0.00 -> 56.9 mm, vias 0 -> 2
- net +3V3: track 0.00 -> 56.0 mm, vias 0 -> 20
- net I2C1_SCL: track 0.00 -> 53.3 mm, vias 0 -> 1
- net SWO: track 0.00 -> 49.3 mm
- net SWDIO: track 0.00 -> 46.1 mm
- net SWCLK: track 0.00 -> 44.9 mm
- net PC13: track 0.00 -> 41.9 mm, vias 0 -> 1
- net PC8: track 0.00 -> 41.7 mm, vias 0 -> 1
- net PC15: track 0.00 -> 40.8 mm, vias 0 -> 1
- net PA4: track 0.00 -> 40.0 mm, vias 0 -> 1
- net PC14: track 0.00 -> 39.9 mm, vias 0 -> 1
- net PA5: track 0.00 -> 38.2 mm, vias 0 -> 1
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- added copper zone on In2.Cu, net +3V3
- added copper zone on In1.Cu, net GND
Other:
- board outline added: 99.6 x 65.1 mm
- board text added: "12V"
- board text added: "3V3"
- board text added: "5V"
- board text added: "Astromech Board 1.3"
- board text added: "BOOT"
- board text added: "Darren Chiu"
- board text added: "GND"
- board text added: "JLCJLCJLCJLC"
- board text added: "PA10"
- board text added: "PA4"
- board text added: "PA5"
- board text added: "PA6"
- board text added: "PA7"
- board text added: "PA8"
- board text added: "PA9"
- board text added: "PB0"
- board text added: "PB1"
- board text added: "PB2"
- board text added: "PC13"
- board text added: "PC14"
- board text added: "PC15"
- board text added: "PC4"
- board text added: "PC5"
- board text added: "PC6"
- board text added: "PC7"
- board text added: "PC8"
- board text added: "PC9"
- board text added: "RUN"
- board text added: "RX"
- board text added: "SCL"
- board text added: "SDA"
- board text added: "Status"
- board text added: "TX"
- board text added: "USB"
