File: EVA-02/STMboard.sch (KiCad schematic (older format))
At the start: 30 parts

Commit message: Generated .net files
Parts:
- removed C? (x2): 10u, symbol Device:C_Small
- removed C? (x4): 100nF, symbol Device:C_Small
- removed D?: B5819W, symbol Device:D_Schottky_Small
- removed F?: 500mA, symbol Device:Fuse
- removed FB?: 100 @ 100MHz, symbol Device:Ferrite_Bead_Small
- removed J?: Conn_02x05_Odd_Even, symbol Connector_Generic:Conn_02x05_Odd_Even
- removed R? (x2): 10k, symbol Device:R_Small
- removed U?: AMS1117-3.3, Package_TO_SOT_SMD:SOT-223-3_TabPin2, symbol Regulator_Linear:AMS1117-3.3
- added C10, C11: 0.1uF, Capacitor_SMD:C_0603_1608Metric, symbol Device:C_Small
- added C12: 2.2nF, Capacitor_SMD:C_0603_1608Metric, symbol Device:C_Small
- added C13: 10n, Capacitor_SMD:C_0201_0603Metric, symbol Device:C_Small
- added C14, C15, C7: 10u, Capacitor_SMD:C_1206_3216Metric, symbol Device:C_Small
- added D1: BLUE, LED_SMD:LED_0603_1608Metric, symbol Device:LED_Small
- added D2, D3: B5819W, Diode_SMD:D_SOD-123, symbol Device:D_Schottky_Small
- added D4: RED, LED_SMD:LED_0603_1608Metric, symbol Device:LED_Small
- added F1: 250mA, Fuse:Fuse_1206_3216Metric, symbol Device:Polyfuse_Small
- added FB1: 600 @ 600MHz, Inductor_SMD:L_0805_2012Metric, symbol Device:Ferrite_Bead_Small
- added H1, H2, H3, H4: MountingHole_Pad, MountingHole:MountingHole_4.3mm_M4_Pad_Via, symbol Mechanical:MountingHole_Pad
- added J1: Screw_Terminal_01x02, TerminalBlock_Phoenix:TerminalBlock_Phoenix_PT-1,5-2-3.5-H_1x02_P3.50mm_Horizontal, symbol Connector:Screw_Terminal_01x02
- added J2: USB_B_Micro, Connector_USB:USB_Micro-B_Molex-105017-0001, symbol Connector:USB_B_Micro
- added J3: Conn_02x05_Odd_Even, Connector_PinSocket_1.27mm:PinSocket_2x05_P1.27mm_Vertical_SMD, symbol Connector_Generic:Conn_02x05_Odd_Even
- added J4, J7: Screw_Terminal_01x04, TerminalBlock_Phoenix:TerminalBlock_Phoenix_PT-1,5-4-3.5-H_1x04_P3.50mm_Horizontal, symbol Connector:Screw_Terminal_01x04
- added J5, J8: Screw_Terminal_01x05, TerminalBlock_Phoenix:TerminalBlock_Phoenix_PT-1,5-5-3.5-H_1x05_P3.50mm_Horizontal, symbol Connector:Screw_Terminal_01x05
- added J6: Screw_Terminal_01x11, TerminalBlock_Phoenix:TerminalBlock_Phoenix_PT-1,5-11-3.5-H_1x11_P3.50mm_Horizontal, symbol Connector:Screw_Terminal_01x11
- added L1: 10u, Inductor_SMD:L_Sunlord_MWSA0518_5.4x5.2mm, symbol Device:L_Small
- added Q1: AO3401A, Package_TO_SOT_SMD:SOT-23, symbol Transistor_FET:AO3401A
- added R1: 1k5, Resistor_SMD:R_0603_1608Metric, symbol Device:R_Small
- added R10: 1k, Resistor_SMD:R_0603_1608Metric, symbol Device:R_Small
- added R2: 10k, Resistor_SMD:R_0402_1005Metric, symbol Device:R_Small
- added R3: 100k, Resistor_SMD:R_0603_1608Metric, symbol Device:R_Small
- added R4: 68k, Resistor_SMD:R_0603_1608Metric, symbol Device:R_Small
- added R5, R6: 2k2, Resistor_SMD:R_0402_1005Metric, symbol Device:R_Small
- added R7: 47k, Resistor_SMD:R_0603_1608Metric, symbol Device:R_Small
- added R8: 15k, Resistor_SMD:R_0603_1608Metric, symbol Device:R_Small
- added R9: 270, Resistor_SMD:R_0603_1608Metric, symbol Device:R_Small
- added SW1: SW_SPDT, Button_Switch_SMD:SW_SPDT_PCM12, symbol Switch:SW_SPDT
- added U2: MP2359DJ-LF-Z, Package_TO_SOT_SMD:SOT-23-6, symbol darren-library:MP2359DJ-LF-Z
- added U4: USBLC6-2SC6, Package_TO_SOT_SMD:SOT-23-6, symbol Power_Protection:USBLC6-2SC6
- added U5, U6: ULN2003A, Package_SO:SOIC-16_3.9x9.9mm_P1.27mm, symbol Transistor_Array:ULN2003A
- C1: renamed from C?; value 10u -> 4u7; footprint (none) -> Capacitor_SMD:C_0603_1608Metric
- C16, C17, C19: renamed from C?; footprint (none) -> Capacitor_SMD:C_0402_1005Metric
- C18: renamed from 12p; value C_Small -> 12p; footprint (none) -> Capacitor_SMD:C_0402_1005Metric
- C2, C3, C4, C5, C6, C8, C9: renamed from C?; footprint (none) -> Capacitor_SMD:C_0603_1608Metric
- FB2: renamed from FB?; footprint (none) -> Inductor_SMD:L_0805_2012Metric
- HSE1: renamed from HSE; footprint (none) -> Crystal:Crystal_SMD_3225-4Pin_3.2x2.5mm
- R11: renamed from R?; value 120 -> 47; footprint (none) -> Resistor_SMD:R_0402_1005Metric
- gave numbers to parts that had none: 2
Connections:
- net +3V3: now also U3.13 (VDD), U3.8 (VDDIO), C10.1, C14.1, C15.1, D4.2 (A), J3.1 (Pin_1), J4.1 (Pin_1), J6.1 (Pin_1), J7.1 (Pin_1), L1.2, R5.2, R6.2, R7.2, SW1.1 (A)
- net BOOT0: now also R2.2
- net GND: now also U3.1 (CLKIN), U3.11 (FSYNC), U3.18 (GND), U3.9 (AD0), C10.2, C11.2, C12.2, C14.2, C15.2, C7.2, D3.2 (A), H1.1, H2.1, H3.1, H4.1, J1.2 (Pin_2), J2.5 (GND), J3.3 (Pin_3), J3.5 (Pin_5), J3.9 (Pin_9), J4.4 (Pin_4), J6.11 (Pin_11), J7.4 (Pin_4), Q1.1 (G), R1.2, R10.1, R4.1, R9.1, SW1.3 (C), U2.2 (GND), U4.2 (GND), U5.8 (GND), U6.8 (GND); no longer C16.1, HSE1.1, U1.5 (PH0)
- net NRST: now also J3.10 (Pin_10)
- net SWCLK: now also J3.4 (Pin_4)
- net SWDIO: now also J3.2 (Pin_2)
- net SWO: now also J3.6 (Pin_6)
- net at U3.10 (REGOUT): now also C11.1
- net at U3.20 (CPOUT): now also C12.1
- net I2C1_SCL: now reaches U3.23 (SCL)
- net I2C1_SCL: now also U1.58 (PB6), J4.2 (Pin_2), R5.1
- net I2C1_SDA: now reaches U3.24 (SDA)
- net I2C1_SDA: now also U1.59 (PB7), J4.3 (Pin_3), R6.1
- net LED_STATUS: now reaches U1.16 (PA2)
- net LED_STATUS: now also D1.2 (A)
- net PA4: now reaches U1.20 (PA4)
- net PA4: now also J6.2 (Pin_2)
- net PA5: now reaches U1.21 (PA5)
- net PA5: now also J6.3 (Pin_3)
- net PA6: now reaches U1.22 (PA6)
- net PA6: now also J6.4 (Pin_4)
- net PA7: now reaches U1.23 (PA7)
- net PA7: now also J6.5 (Pin_5)
- net PC4: now reaches U1.24 (PC4)
- net PC4: now also J6.6 (Pin_6)
- net PC5: now reaches U1.25 (PC5)
- net PC5: now also J6.7 (Pin_7)
- net PB0: now reaches U1.26 (PB0)
- net PB0: now also J6.8 (Pin_8)
- net PB1: now reaches U1.27 (PB1)
- net PB1: now also J6.9 (Pin_9)
- net UART3_TX: now reaches U1.29 (PB10)
- net UART3_TX: now also J7.2 (Pin_2)
- net UART3_RX: now reaches U1.30 (PB11)
- net UART3_RX: now also J7.3 (Pin_3)
- net STEP_2-4: now reaches U1.36 (PB15)
- net STEP_2-4: now also U6.4 (I4)
- net STEP_2-3: now reaches U1.37 (PC6)
- net STEP_2-3: now also U6.3 (I3)
- net STEP_2-2: now reaches U1.38 (PC7)
- net STEP_2-2: now also U6.2 (I2)
- net STEP_2-1: now reaches U1.39 (PC8)
- net STEP_2-1: now also U6.1 (I1)
- net STEP_1-4: now reaches U1.40 (PC9)
- net STEP_1-4: now also U5.4 (I4)
- net STEP_1-3: now reaches U1.41 (PA8)
- net STEP_1-3: now also U5.3 (I3)
- net STEP_1-2: now reaches U1.42 (PA9)
- net STEP_1-2: now also U5.2 (I2)
- net STEP_1-1: now reaches U1.43 (PA10)
- net STEP_1-1: now also U5.1 (I1)
- net USB_D-: now reaches U1.44 (PA11)
- net USB_D-: now also U4.6 (I/O1)
- net USB_D+: now reaches U1.45 (PA12)
- net USB_D+: now also U4.4 (I/O2)
- net BOOT1 renamed PB2
- net PB2: now also J6.10 (Pin_10)
- new net: R2.1, SW1.2 (B)
- new net: D1.1 (K), R1.1
- new net: J5.4 (Pin_4), U5.13 (O4)
- new net: J5.3 (Pin_3), U5.14 (O3)
- new net: J5.2 (Pin_2), U5.15 (O2)
- new net: J5.1 (Pin_1), U5.16 (O1)
- new net: J8.4 (Pin_4), U6.13 (O4)
- new net: J8.3 (Pin_3), U6.14 (O3)
- new net: J8.2 (Pin_2), U6.15 (O2)
- new net: J8.1 (Pin_1), U6.16 (O1)
- new net: F1.1, Q1.3 (D)
- new net: D2.1 (K), FB1.2, Q1.2 (S)
- new net: R8.1, R9.2
- new net: D4.1 (K), R10.2
- new net +12V: F1.2, J1.1 (Pin_1)
- new net +5V: D2.2 (A), J2.1 (VBUS), J5.5 (Pin_5), J8.5 (Pin_5), U4.5 (VBUS)
- new net BUCK_BST: C13.1, U2.1 (BST)
- new net BUCK_EN: R3.1, R4.2, U2.4 (EN)
- new net BUCK_FB: R7.1, R8.2, U2.3 (FB)
- new net BUCK_IN: C7.1, FB1.1, R3.2, U2.5 (IN)
- new net BUCK_SW: C13.2, D3.1 (K), L1.1, U2.6 (SW)
- new net HSE_IN: C16.1, HSE1.1, U1.5 (PH0)
- new net USB_CONN_D+: J2.3 (D+), U4.3 (I/O2)
- new net USB_CONN_D-: J2.2 (D-), U4.1 (I/O1)
- no-connect marks 2 -> 43
Other:
- note added: "ADC Filter\n"
- note added: "Decoupling Capacitors\n"
- note added: "Hardware Reset"
- note added: "High Speed External Clock\n"
- moved on the sheet: C1, C16, C17, C18, C19, C2, C3, C4, C5, C6, C8, C9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

Commit message: Manufactured board files
Parts:
- removed FB2: 100 @ 100MHz, Inductor_SMD:L_0805_2012Metric, symbol Device:Ferrite_Bead_Small
- removed J1: Screw_Terminal_01x02, TerminalBlock_Phoenix:TerminalBlock_Phoenix_PT-1,5-2-3.5-H_1x02_P3.50mm_Horizontal, symbol Connector:Screw_Terminal_01x02
- added J1: Screw_Terminal_01x06, TerminalBlock_Phoenix:TerminalBlock_Phoenix_PT-1,5-6-3.5-H_1x06_P3.50mm_Horizontal, symbol Connector:Screw_Terminal_01x06
- added L2: 39n, Inductor_SMD:L_0402_1005Metric, symbol Device:L_Small
- C1: LCSC Part # (none) -> C19666
- C10, C11: value 0.1uF -> 100nF; LCSC Part # (none) -> C14663
- C12: LCSC Part # (none) -> C1604
- C13: footprint Capacitor_SMD:C_0201_0603Metric -> Capacitor_SMD:C_0402_1005Metric; LCSC Part # (none) -> C15195
- C14, C15, C16, C18, C7: LCSC Part # (none) -> C13585
- C17: value 100nF -> 1u; LCSC Part # (none) -> C1525
- C19: LCSC Part # (none) -> C15195
- C2, C4: LCSC Part # (none) -> C23630
- C3, C5, C6, C8, C9: LCSC Part # (none) -> C14663
- D1: LCSC Part # (none) -> C72041
- D2, D3: LCSC Part # (none) -> C8598
- D4: LCSC Part # (none) -> C2286
- F1: LCSC Part # (none) -> C369159
- FB1: LCSC Part # (none) -> C1017
- HSE1: LCSC Part # (none) -> C13738
- J3: footprint Connector_PinSocket_1.27mm:PinSocket_2x05_P1.27mm_Vertical_SMD -> Connector_PinHeader_1.27mm:PinHeader_2x05_P1.27mm_Vertical_SMD
- L1: LCSC Part # (none) -> C139506
- Q1: LCSC Part # (none) -> C15127
- R1: LCSC Part # (none) -> C22843
- R10: LCSC Part # (none) -> C21190
- R11: LCSC Part # (none) -> C25118
- R2: LCSC Part # (none) -> C25744
- R3: LCSC Part # (none) -> C25803
- R4: LCSC Part # (none) -> C23231
- R5, R6: LCSC Part # (none) -> C25879
- R7: LCSC Part # (none) -> C25819
- R8: LCSC Part # (none) -> C22809
- R9: LCSC Part # (none) -> C22966
- U1: LCSC Part # (none) -> C15742
- U2: LCSC Part # (none) -> C14259
- U3: LCSC Part # (none) -> C24112
- U4: LCSC Part # (none) -> C7519
- U5, U6: LCSC Part # (none) -> C7512
Connections:
- net +12V: now also J1.1 (Pin_1)
- net +3.3VA: now also L2.2
- net +3V3: now also L2.1
- net +5V: now also J5.1 (Pin_1), J8.1 (Pin_1); no longer J5.5 (Pin_5), J8.5 (Pin_5)
- net GND: now also J1.2 (Pin_2)
- net PC13: now reaches U1.2 (PC13)
- net PC13: now also J1.3 (Pin_3)
- net PC14: now reaches U1.3 (PC14)
- net PC14: now also J1.4 (Pin_4)
- net PC15: now reaches U1.4 (PC15)
- net PC15: now also J1.5 (Pin_5)
- net PC8: now reaches U1.8 (PC0)
- net PC8: now also J1.6 (Pin_6)
- net at U5.13 (O4): now also J5.2 (Pin_2); no longer J5.4 (Pin_4)
- net at U5.15 (O2): now also J5.4 (Pin_4); no longer J5.2 (Pin_2)
- net at U5.16 (O1): now also J5.5 (Pin_5); no longer J5.1 (Pin_1)
- net at U6.13 (O4): now also J8.2 (Pin_2); no longer J8.4 (Pin_4)
- net at U6.15 (O2): now also J8.4 (Pin_4); no longer J8.2 (Pin_2)
- net at U6.16 (O1): now also J8.5 (Pin_5); no longer J8.1 (Pin_1)
- no-connect marks 43 -> 39
Other:
- moved on the sheet: J5, J8, U6
