File: Astromech3.0/Astromech3.0.sch (KiCad schematic (older format))
At the start: 48 parts, among them J1 Screw_Terminal_01x02, J2 Conn_01x04, J3 USB_B_Micro, J4 Conn_01x03_Male, J5 Conn_01x05, SW1 SW_Push, SW2 SW_Push, U1 STM32F103C8Tx, U2 MPU-6050, U3 AMS1117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

Commit message: final manufactured board
Parts:
- removed C11, C14: 100uF, Capacitor_SMD:C_0603_1608Metric, symbol Device:CP1_Small
- removed J2: Conn_01x04, Connector_PinHeader_1.27mm:PinHeader_1x04_P1.27mm_Vertical, symbol Connector_Generic:Conn_01x04
- removed J4: Conn_01x03_Male, Connector_PinHeader_1.27mm:PinHeader_1x03_P1.27mm_Vertical, symbol Connector:Conn_01x03_Male
- removed J5: Conn_01x05, Connector_PinHeader_1.27mm:PinHeader_1x05_P1.27mm_Vertical, symbol Connector_Generic:Conn_01x05
- added C11: 100nF, Capacitor_SMD:C_0402_1005Metric, symbol Device:C_Small
- added J2: Conn_01x02, Connector_PinHeader_1.27mm:PinHeader_1x02_P1.27mm_Vertical, symbol Connector_Generic:Conn_01x02
- added J4: Conn_01x04, Connector_PinHeader_1.27mm:PinHeader_1x04_P1.27mm_Vertical, symbol Connector_Generic:Conn_01x04
- added J5: Conn_01x07, Connector_PinHeader_1.27mm:PinHeader_1x07_P1.27mm_Vertical, symbol Connector_Generic:Conn_01x07
- added J6: Conn_01x06, Connector_PinHeader_1.27mm:PinHeader_1x06_P1.27mm_Vertical, symbol Connector_Generic:Conn_01x06
- C1, C10, C4, C5, C6, C7, C9: LCSC Part # (none) -> C1525
- C12: footprint Capacitor_SMD:C_0603_1608Metric -> Capacitor_SMD:C_0402_1005Metric; LCSC Part # (none) -> C1525
- C13, C15, C18, C19: footprint Capacitor_SMD:C_0603_1608Metric -> Capacitor_SMD:C_0402_1005Metric; LCSC Part # (none) -> C361198
- C16: LCSC Part # (none) -> C1604
- C17: value 100nF -> 10uF; footprint Capacitor_SMD:C_0603_1608Metric -> Capacitor_SMD:C_0402_1005Metric; LCSC Part # (none) -> C15525
- C2, C3: LCSC Part # (none) -> C38523
- C8: value 1uF -> 10uF; footprint Capacitor_SMD:C_01005_0402Metric -> Capacitor_SMD:C_0402_1005Metric; LCSC Part # (none) -> C15525
- D1: LCSC Part # (none) -> C2286
- D2: LCSC Part # (none) -> C72038
- D3: LCSC Part # (none) -> C72043
- H1, H2, H3, H4: footprint MountingHole:MountingHole_2.7mm_M2.5 -> MountingHole:MountingHole_2.2mm_M2_DIN965_Pad
- J3: LCSC Part # (none) -> C10418
- R1, R2, R3, R4: LCSC Part # (none) -> C25744
- R10, R6, R7: LCSC Part # (none) -> C23193
- R5: LCSC Part # (none) -> C17557
- R8, R9: LCSC Part # (none) -> C1532
- U1: LCSC Part # (none) -> C8734
- U2: LCSC Part # (none) -> C24112
- U3: LCSC Part # (none) -> C6186
- U4: LCSC Part # (none) -> C97521
- Y1: LCSC Part # (none) -> C13738
Connections:
- net PA4 is gone; now on net QSPI_CS: U1.14 (PA4)
- net PA5 is gone; now on net QSPI_CLK: U1.15 (PA5)
- net +3V3: now also C11.1, J4.1 (Pin_1); no longer C8.1
- net +5V: now also C8.1
- net GND: now also C11.2, J4.4 (Pin_4)
- net QSPI_CLK: no longer U1.26 (PB13)
- net QSPI_CS: no longer U1.25 (PB12)
- net SWCLK: now also J2.2 (Pin_2)
- net SWDIO: now also J2.1 (Pin_1)
- net UART_RX: now also J4.3 (Pin_3)
- net UART_TX: now also J4.2 (Pin_2)
- net PB0: now reaches U1.18 (PB0)
- net PB1: now reaches U1.19 (PB1)
- net PB2: now reaches U1.20 (PB2)
- net PA10: now reaches U1.31 (PA10)
- net PA10: now also J5.1 (Pin_1)
- net PA15: now reaches U1.38 (PA15)
- net PA15: now also J6.1 (Pin_1)
- net PB3: now reaches U1.39 (PB3)
- net PB3: now also J6.2 (Pin_2)
- net PB4: now reaches U1.40 (PB4)
- net PB4: now also J6.3 (Pin_3)
- net PB5: now reaches U1.41 (PB5)
- net PB5: now also J6.4 (Pin_4)
- net PB8: now reaches U1.45 (PB8)
- net PB8: now also J6.5 (Pin_5)
- net PB9: now reaches U1.46 (PB9)
- net PB9: now also J6.6 (Pin_6)
- net PA3: no longer names the net of U1.13 (PA3)
- net PA6 renamed SPI_MISO
- net SPI_MISO: now also U4.5 (DI(IO0))
- net PA7 renamed SPI_MOSI
- net SPI_MOSI: now also U4.2 (DO(IO1))
- net QSPI_IO0 renamed PA9
- net PA9: now also J5.2 (Pin_2); no longer U4.5 (DI(IO0))
- net QSPI_IO1 renamed PA8
- net PA8: now also J5.3 (Pin_3); no longer U4.2 (DO(IO1))
- net QSPI_IO2: no longer names the net of U4.3 (IO2)
- net QSPI_IO2: no longer U1.28 (PB15)
- net QSPI_IO3: no longer names the net of U4.7 (IO3)
- net QSPI_IO3: no longer U1.27 (PB14)
- new net PB12: J5.7 (Pin_7), U1.25 (PB12)
- new net PB13: J5.6 (Pin_6), U1.26 (PB13)
- new net PB14: J5.5 (Pin_5), U1.27 (PB14)
- new net PB15: J5.4 (Pin_4), U1.28 (PB15)
- no-connect marks 5 -> 6
